File: hardware/hard tp/hard tp.kicad_sch (KiCad schematic)
At the start: 11 parts, among them U1 STM32L021K4T6

Commit message: modif final séance 1
Parts:
- added C10: 10u, Capacitor_SMD:C_0805_2012Metric, symbol Device:C
- added C7, C8: 1uF, Capacitor_SMD:C_0805_2012Metric, symbol Device:C
- added C9: 100n, Capacitor_SMD:C_0805_2012Metric_Pad1.18x1.45mm_HandSolder, symbol Device:C
- added D2: GREEN LED, LED_SMD:LED_0603_1608Metric_Pad1.05x0.95mm_HandSolder, symbol Device:LED
- added J1: Conn_02x07_Odd_Even, Connector_PinHeader_1.27mm:PinHeader_2x07_P1.27mm_Vertical_SMD, symbol Connector_Generic:Conn_02x07_Odd_Even
- added J2, J3, J4: Conn_01x02, Connector_JST:JST_XH_B2B-XH-A_1x02_P2.50mm_Vertical, symbol Connector_Generic:Conn_01x02
- added R3: 1k, Resistor_SMD:R_0805_2012Metric_Pad1.20x1.40mm_HandSolder, symbol Device:R
- added U2: MCP4801, Package_SO:SOIC-8_3.9x4.9mm_P1.27mm, symbol Analog_DAC:MCP4801
- added U3: BU33SD5WG-TR, Package_TO_SOT_SMD:SOT-23-5, symbol Regulator_Linear:MCP1802x-xx02xOT
- C1, C2, C3, C5: footprint (none) -> Capacitor_SMD:C_0805_2012Metric_Pad1.18x1.45mm_HandSolder
- C4: renamed from C10; footprint (none) -> Capacitor_SMD:C_0805_2012Metric_Pad1.18x1.45mm_HandSolder
- C6: renamed from C7; footprint (none) -> Capacitor_SMD:C_0805_2012Metric_Pad1.18x1.45mm_HandSolder
- D1: footprint (none) -> LED_SMD:LED_0603_1608Metric_Pad1.05x0.95mm_HandSolder
- L1: footprint (none) -> Inductor_SMD:L_0805_2012Metric_Pad1.05x1.20mm_HandSolder
- R1: footprint (none) -> Resistor_SMD:R_0805_2012Metric_Pad1.20x1.40mm_HandSolder
- R2: renamed from R3; footprint (none) -> Resistor_SMD:R_0805_2012Metric_Pad1.20x1.40mm_HandSolder
Connections:
- net +3.3V: now also C8.1, D2.2 (A), J1.3 (Pin_3), U3.5 (VOUT)
- net +3.3VA: now also C10.1, C9.1, U2.1 (Vdd), U2.6 (~{SHDN})
- net ADC_IN1: now also J2.1 (Pin_1)
- net DAC_nCS: now also U2.2 (~{CS})
- net GND: now also C10.2, C7.2, C8.2, C9.2, J1.11 (Pin_11), J1.5 (Pin_5), J1.7 (Pin_7), J2.2 (Pin_2), J3.2 (Pin_2), J4.2 (Pin_2), R3.2, U2.7 (Vss), U3.2 (GND)
- net SPI1_SCK: now also U2.3 (SCK)
- net SWDCK: now also J1.6 (Pin_6)
- net SWDIO: now also J1.4 (Pin_4)
- net USART2_RX: now also J1.13 (Pin_13)
- net USART2_TX: now also J1.14 (Pin_14)
- net DAC-nLDAC renamed DAC_nLDAC
- net DAC_nLDAC: now also U2.5 (~{LDAC})
- net SPI_MOSI renamed SPI1_MOSI
- net SPI1_MOSI: now also U2.4 (SDI)
- new net: D2.1 (K), R3.1
- new net +5V: C7.1, J3.1 (Pin_1), U3.1 (VIN), U3.3 (~{SHDN})
- new net DAC_OUT: J4.1 (Pin_1), U2.8 (Vout)
- new net NRST: J1.12 (Pin_12)
- no-connect marks 15 -> 20

Commit message: readme
Parts:
- added H1, H2, H3, H4: MountingHole_Pad, MountingHole:MountingHole_3.2mm_M3_Pad, symbol Mechanical:MountingHole_Pad
Connections:
- net NSRT is gone; now on net NRST: C4.1, U1.4 (NRST)
- net GND: now also H1.1, H2.1, H3.1, H4.1
Changed lines of the file:
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@@
   (junction (at 152.4 38.1) (diameter 0) (color 0 0 0 0)
   )
+  (junction (at 38.1 60.96) (diameter 0) (color 0 0 0 0)
+  )
   (junction (at 212.09 46.99) (diameter 0) (color 0 0 0 0)
   )
+  (junction (at 38.1 54.61) (diameter 0) (color 0 0 0 0)
+  )
   (junction (at 161.29 27.94) (diameter 0) (color 0 0 0 0)
   )
@@
   )
   (junction (at 87.63 40.64) (diameter 0) (color 0 0 0 0)
+  )
+  (junction (at 38.1 48.26) (diameter 0) (color 0 0 0 0)
   )
   (junction (at 87.63 33.02) (diameter 0) (color 0 0 0 0)
@@
     (stroke (width 0) (type default) (color 0 0 0 0))
   )
+  (wire (pts (xy 38.1 60.96) (xy 44.45 60.96))
+    (stroke (width 0) (type default) (color 0 0 0 0))
+  )
   (wire (pts (xy 152.4 38.1) (xy 161.29 38.1))
     (stroke (width 0) (type default) (color 0 0 0 0))
@@
     (stroke (width 0) (type default) (color 0 0 0 0))
   )
+  (wire (pts (xy 38.1 41.91) (xy 38.1 48.26))
+    (stroke (width 0) (type default) (color 0 0 0 0))
+  )
   (wire (pts (xy 152.4 86.36) (xy 151.13 86.36))
     (stroke (width 0) (type default) (color 0 0 0 0))
@@
     (stroke (width 0) (type default) (color 0 0 0 0))
   )
+  (wire (pts (xy 38.1 48.26) (xy 38.1 54.61))
+    (stroke (width 0) (type default) (color 0 0 0 0))
+  )
   (wire (pts (xy 203.2 30.48) (xy 203.2 33.02))
     (stroke (width 0) (type default) (color 0 0 0 0))
@@
     (stroke (width 0) (type default) (color 0 0 0 0))
   )
+  (wire (pts (xy 38.1 48.26) (xy 44.45 48.26))
+    (stroke (width 0) (type default) (color 0 0 0 0))
+  )
   (wire (pts (xy 139.7 109.22) (xy 138.43 109.22))
     (stroke (width 0) (type default) (color 0 0 0 0))
@@
     (stroke (width 0) (type default) (color 0 0 0 0))
   )
+  (wire (pts (xy 44.45 41.91) (xy 38.1 41.91))
+    (stroke (width 0) (type default) (color 0 0 0 0))
+  )
   (wire (pts (xy 113.03 74.93) (xy 113.03 73.66))
     (stroke (width 0) (type default) (color 0 0 0 0))
@@
     (stroke (width 0) (type default) (color 0 0 0 0))
   )
+  (wire (pts (xy 38.1 54.61) (xy 44.45 54.61))
+    (stroke (width 0) (type default) (color 0 0 0 0))
+  )
   (wire (pts (xy 248.92 30.48) (xy 248.92 33.02))
     (stroke (width 0) (type default) (color 0 0 0 0))
@@
     (stroke (width 0) (type default) (color 0 0 0 0))
   )
+  (wire (pts (xy 38.1 54.61) (xy 38.1 60.96))
+    (stroke (width 0) (type default) (color 0 0 0 0))
+  )
   (wire (pts (xy 212.09 46.99) (xy 227.33 46.99))
     (stroke (width 0) (type default) (color 0 0 0 0))
@@
   )
   (wire (pts (xy 139.7 109.22) (xy 139.7 113.03))
+    (stroke (width 0) (type default) (color 0 0 0 0))
+  )
+  (wire (pts (xy 38.1 60.96) (xy 38.1 66.04))
     (stroke (width 0) (type default) (color 0 0 0 0))
   )
@@
     )
   )
-  (global_label "NSRT" (shape input) (at 111.76 66.04 180) (fields_autoplaced)
+  (global_label "LED_STATUS" (shape input) (at 100.33 97.79 90) (fields_autoplaced)
+    (effects (font (size 1.27 1.27)) (justify left))
+    (property "Références Inter-Feuilles" "${INTERSHEET_REFS}" (id 0) (at 100.2506 84.1888 90)
+      (effects (font (size 1.27 1.27)) (justify left) hide)
+    )
+  )
+  (global_label "SWDIO" (shape input) (at 152.4 99.06 0) (fields_autoplaced)
+    (effects (font (size 1.27 1.27)) (justify left))
+    (property "Références Inter-Feuilles" "${INTERSHEET_REFS}" (id 0) (at 160.6793 98.9806 0)
+      (effects (font (size 1.27 1.27)) (justify left) hide)
+    )
+  )
+  (global_label "NRST" (shape input) (at 111.76 66.04 180) (fields_autoplaced)
     (effects (font (size 1.27 1.27)) (justify right))
-    (property "Références Inter-Feuilles" "${INTERSHEET_REFS}" (id 0) (at 104.5693 65.9606 0)
+    (property "Références Inter-Feuilles" "${INTERSHEET_REFS}" (id 0) (at 104.5693 66.1194 0)
       (effects (font (size 1.27 1.27)) (justify right) hide)
-    )
-  )
-  (global_label "LED_STATUS" (shape input) (at 100.33 97.79 90) (fields_autoplaced)
-    (effects (font (size 1.27 1.27)) (justify left))
-    (property "Références Inter-Feuilles" "${INTERSHEET_REFS}" (id 0) (at 100.2506 84.1888 90)
-      (effects (font (size 1.27 1.27)) (justify left) hide)
-    )
-  )
-  (global_label "SWDIO" (shape input) (at 152.4 99.06 0) (fields_autoplaced)
-    (effects (font (size 1.27 1.27)) (justify left))
-    (property "Références Inter-Feuilles" "${INTERSHEET_REFS}" (id 0) (at 160.6793 98.9806 0)
-      (effects (font (size 1.27 1.27)) (justify left) hide)
     )
   )
@@
     (pin "1")
   )
+  (symbol (lib_id "Mechanical:MountingHole_Pad") (at 46.99 60.96 270) (unit 1)
+    (in_bom yes) (on_board yes) (fields_autoplaced)
+    (property "Reference" "H4" (id 0) (at 50.8 59.6899 90)
+      (effects (font (size 1.27 1.27)) (justify left))
+    )
+    (property "Value" "MountingHole_Pad" (id 1) (at 50.8 62.2299 90)
+      (effects (font (size 1.27 1.27)) (justify left))
+    )
+    (property "Footprint" "MountingHole:MountingHole_3.2mm_M3_Pad" (id 2) (at 46.99 60.96 0)
+      (effects (font (size 1.27 1.27)) hide)
+    )
+    (property "Datasheet" "~" (id 3) (at 46.99 60.96 0)
+      (effects (font (size 1.27 1.27)) hide)
+    )
+    (pin "1")
+  )
   (symbol (lib_id "power:+3.3V") (at 87.63 27.94 0) (unit 1)
     (in_bom yes) (on_board yes) (fields_autoplaced)
@@
     (pin "1")
   )
+  (symbol (lib_id "Mechanical:MountingHole_Pad") (at 46.99 54.61 270) (unit 1)
+    (in_bom yes) (on_board yes) (fields_autoplaced)
+    (property "Reference" "H3" (id 0) (at 50.8 53.3399 90)
+      (effects (font (size 1.27 1.27)) (justify left))
+    )
+    (property "Value" "MountingHole_Pad" (id 1) (at 50.8 55.8799 90)
+      (effects (font (size 1.27 1.27)) (justify left))
+    )
+    (property "Footprint" "MountingHole:MountingHole_3.2mm_M3_Pad" (id 2) (at 46.99 54.61 0)
+      (effects (font (size 1.27 1.27)) hide)
+    )
+    (property "Datasheet" "~" (id 3) (at 46.99 54.61 0)
+      (effects (font (size 1.27 1.27)) hide)
+    )
+    (pin "1")
+  )
   (symbol (lib_id "power:GND") (at 240.03 129.54 0) (unit 1)
     (in_bom yes) (on_board yes) (fields_autoplaced)
@@
     (pin "1")
   )
+  (symbol (lib_id "Mechanical:MountingHole_Pad") (at 46.99 48.26 270) (unit 1)
+    (in_bom yes) (on_board yes) (fields_autoplaced)
+    (property "Reference" "H2" (id 0) (at 50.8 46.9899 90)
+      (effects (font (size 1.27 1.27)) (justify left))
+    )
+    (property "Value" "MountingHole_Pad" (id 1) (at 50.8 49.5299 90)
+      (effects (font (size 1.27 1.27)) (justify left))
+    )
+    (property "Footprint" "MountingHole:MountingHole_3.2mm_M3_Pad" (id 2) (at 46.99 48.26 0)
+      (effects (font (size 1.27 1.27)) hide)
+    )
+    (property "Datasheet" "~" (id 3) (at 46.99 48.26 0)
+      (effects (font (size 1.27 1.27)) hide)
+    )
+    (pin "1")
+  )
   (symbol (lib_id "Device:C") (at 87.63 36.83 0) (unit 1)
     (in_bom yes) (on_board yes) (fields_autoplaced)
@@
     (pin "1")
     (pin "2")
+  )
+  (symbol (lib_id "power:GND") (at 38.1 66.04 0) (unit 1)
+    (in_bom yes) (on_board yes) (fields_autoplaced)
+    (property "Reference" "#PWR0101" (id 0) (at 38.1 72.39 0)
+      (effects (font (size 1.27 1.27)) hide)
+    )
+    (property "Value" "GND" (id 1) (at 38.1 71.12 0))
+    (property "Footprint" "" (id 2) (at 38.1 66.04 0)
+      (effects (font (size 1.27 1.27)) hide)
+    )
+    (property "Datasheet" "" (id 3) (at 38.1 66.04 0)
+      (effects (font (size 1.27 1.27)) hide)
+    )
+    (pin "1")
   )
   (symbol (lib_id "power:GND") (at 113.03 74.93 0) (unit 1)
@@
     (pin "1")
   )
+  (symbol (lib_id "Mechanical:MountingHole_Pad") (at 46.99 41.91 270) (unit 1)
+    (in_bom yes) (on_board yes) (fields_autoplaced)
+    (property "Reference" "H1" (id 0) (at 50.8 40.6399 90)
+      (effects (font (size 1.27 1.27)) (justify left))
+    )
+    (property "Value" "MountingHole_Pad" (id 1) (at 50.8 43.1799 90)
+      (effects (font (size 1.27 1.27)) (justify left))
+    )
+    (property "Footprint" "MountingHole:MountingHole_3.2mm_M3_Pad" (id 2) (at 46.99 41.91 0)
+      (effects (font (size 1.27 1.27)) hide)
+    )
+    (property "Datasheet" "~" (id 3) (at 46.99 41.91 0)
+      (effects (font (size 1.27 1.27)) hide)
+    )
+    (pin "1")
+  )
   (symbol (lib_id "Device:C") (at 147.32 34.29 0) (unit 1)
     (in_bom yes) (on_board yes) (fields_autoplaced)
@@
       (reference "#PWR025") (unit 1) (value "GND") (footprint "")
     )
+    (path "/b94c633e-98b9-4128-b026-b044f6934f6f"
+      (reference "#PWR0101") (unit 1) (value "GND") (footprint "")
+    )
     (path "/9867df9f-c114-472a-82e2-73a7025b9300"
       (reference "C1") (unit 1) (value "4u7") (footprint "Capacitor_SMD:C_0805_2012Metric_Pad1.18x1.45mm_HandSolder")
@@
       (reference "D2") (unit 1) (value "GREEN LED") (footprint "LED_SMD:LED_0603_1608Metric_Pad1.05x0.95mm_HandSolder")
     )
+    (path "/faeed6ba-591a-41e6-aad3-a25da02740c9"
+      (reference "H1") (unit 1) (value "MountingHole_Pad") (footprint "MountingHole:MountingHole_3.2mm_M3_Pad")
+    )
+    (path "/96b2e68b-f0a3-4b8b-a9ec-d531fe048f20"
+      (reference "H2") (unit 1) (value "MountingHole_Pad") (footprint "MountingHole:MountingHole_3.2mm_M3_Pad")
+    )
+    (path "/65e6473a-faeb-458d-bbae-cc43b9088d34"
+      (reference "H3") (unit 1) (value "MountingHole_Pad") (footprint "MountingHole:MountingHole_3.2mm_M3_Pad")
+    )
+    (path "/4dbb2a00-c361-4ebd-88e8-aa989d02985d"
+      (reference "H4") (unit 1) (value "MountingHole_Pad") (footprint "MountingHole:MountingHole_3.2mm_M3_Pad")
+    )
     (path "/34b9ccac-7762-4783-ac5d-fbba7c98d3c7"
